File: ambient-air.kicad_sch (KiCad schematic)
At the start: 23 parts, among them J5 USB_C_Receptacle_USB2.0_14P, U1 AP7361C-33SP-13, U2 MCP73831-2-MC, U3 ESP32-C3-WROOM-02, U4 AHT20_C2757850, U5 SGP40-D-R4, U6 ICP-20100, U7 SCCT4-D1

Commit message: Quicksave
Parts:
- added C7, C8: 100nF, Capacitor_SMD:C_0805_2012Metric, symbol Device:C_Small
- added C9: 1µF, Capacitor_SMD:C_0805_2012Metric, symbol Device:C_Small
- added D3, D4: LED, Capacitor_Tantalum_SMD:CP_EIA-3528-12_Kemet-T, symbol Device:LED
- added J2: Conn_01x02, Connector_JST:JST_PH_S2B-PH-SM4-TB_1x02-1MP_P2.00mm_Horizontal, symbol Connector_Generic:Conn_01x02
- added JP1: Jumper_2_Open, Jumper:SolderJumper-2_P1.3mm_Open_TrianglePad1.0x1.5mm, symbol Jumper:Jumper_2_Open
- added R4, R5: 40Ω, Resistor_SMD:R_0603_1608Metric, symbol Device:R_Small
- added R6: 4.7Ω, Resistor_SMD:R_0603_1608Metric, symbol Device:R_Small
- added SW1, SW3: SW_Push, easyeda2kicad:SW-SMD_L6.0-W3.5-LS8.2, symbol Switch:SW_Push
- added SW2: MINI MSK12CO2, easyeda2kicad:SW-SMD_MSK12CO2, symbol easyeda2kicad:MINIMSK12CO2
- added U4: TPD4E05U06DQA, Package_SON:USON-10_2.5x1.0mm_P0.5mm, symbol Power_Protection:TPD4E05U06DQA
- added U5: SHT4x, Sensor_Humidity:Sensirion_DFN-4_1.5x1.5mm_P0.8mm_SHT4x_NoCentralPad, symbol Sensor_Humidity:SHT4x
- C1: footprint (none) -> Capacitor_SMD:C_0805_2012Metric
- C2: renamed from C4; footprint (none) -> Capacitor_SMD:C_0805_2012Metric
- C5: renamed from C2; footprint (none) -> Capacitor_SMD:C_0805_2012Metric
- C6: renamed from C3; footprint (none) -> Capacitor_SMD:C_0805_2012Metric
- D2: renamed from D1; footprint (none) -> Capacitor_Tantalum_SMD:CP_EIA-3528-12_Kemet-T
- R10: renamed from R7; footprint (none) -> Resistor_SMD:R_0805_2012Metric
- R2: renamed from R1; footprint (none) -> Resistor_SMD:R_0805_2012Metric
- R3: renamed from R2; value R_Small -> 100Ω; footprint (none) -> Resistor_SMD:R_0603_1608Metric
- R7: renamed from R4; value 10kΩ -> 12kΩ; footprint Resistor_SMD:R_0805_2012Metric -> Resistor_SMD:R_0603_1608Metric
- R8: renamed from R5; value 5.1kΩ -> 10kΩ; footprint Resistor_SMD:R_0805_2012Metric -> Resistor_SMD:R_0603_1608Metric
- R9: renamed from R8; footprint (none) -> Resistor_SMD:R_0805_2012Metric
- U1: renamed from U2; value MCP73831-2-MC -> MCP73831T-2ACI/MC
- U6: renamed from U7; value SCCT4-D1 -> STCC4-D1; footprint (none) -> easyeda2kicad:STCC4DR3
- U7: renamed from U4; now not fitted
- U8: renamed from U5; footprint SGP40-D-R4:XCDR_SGP40-D-R4 -> easyeda2kicad:XCDR_SGP40-D-R4
- U9: renamed from U6; footprint ICP-20100:PQFN50P200X200X85-10N -> easyeda2kicad:PQFN50P200X200X85-10N
- renumbered C7 to C3, C8 to C4, D2 to D1, J5 to J1, R3 to R1, U1 to U2
Connections:
- net +3V3: now also U6.3 (ADDR), U6.6 (VDDIO), U8.5 (VDDH), U9.1 (CSB), U9.10 (VDDIO), C7.1, C8.1, C9.1, R6.2, U5.3 (VDD); no longer U8.1 (VDD)
- net GND: now also U8.4 (N/A), U8.7 (EXP), U9.6 (SDO/AD0), U9.8 (RESV), U9.9 (RESV), C7.2, C8.2, C9.2, D3.1 (K), D4.1 (K), J2.2 (Pin_2), SW1.1, SW3.1, U4.3 (GND), U4.8 (GND), U5.4 (VSS)
- net SCL: now also U7.3 (SCL)
- net USB_D+: now also U4.1 (D1+)
- net USB_D-: now also U4.2 (D1-)
- net VBAT: now also J2.1 (Pin_1), JP1.2 (B), SW2.3; no longer R7.1
- net VBAT_DIV: now also U3.16 (GPIO2/ADC1_CH2)
- net VBUS: now also D2.2 (A), JP1.1 (A); no longer R3.1
- net at U1.5 (STAT): now also R3.2; no longer D2.1 (K)
- net at U6.2 (SDA_C): now also U5.1 (SDA)
- net at U6.8 (SCL_C): now also U5.2 (SCL)
- net at U3.10 (GPIO10): now also R5.1
- net at U3.15 (GPIO3/ADC1_CH3): now also SW3.2
- net at R1.2, U3.2 (EN/CHIP_PU): now also SW1.2
- net at U3.4 (GPIO5/ADC2_CH0): now also R4.1
- net EN_VBAT: now reaches U2.2 (EN)
- net EN_VBAT: now also R7.1, SW2.2
- new net: R6.1, U8.1 (VDD)
- new net: D4.2 (A), R5.2
- new net: D3.2 (A), R4.2
- new net: D2.1 (K), R3.1
- no-connect marks 7 -> 23
Other:
- note added: "Color: Green Type: QTLP670C-4 IF: 30mA VF: 2.1V"
- note added: "Deep-Sleep: 5µA"
- note added: "I2C Address: 0x38"
- note added: "I2C Address: 0x59"
- note added: "I2C Address: 0x63"
- note added: "I2C Address: 0x65"
- note added: "Sleep: 1µA"
- note added: "Standby: 1µA"
- note added: "Standby: 2.65µA"
- note added: "Standby: 2µA"
- note added: "Standby: 34µA"
- moved on the sheet: D2, R1, R3
