File: Kicad/ambient-air.kicad_pcb (KiCad board)
At the start: 2 copper layers, 50 x 35 mm, 38 parts, among them J1 USB_C_Receptacle_USB2.0_14P, J2 Conn_01x02, SW1 SW_Push, SW2 MINI MSK12CO2, SW3 SW_Push, U1 MCP73831T-2ACI/MC, U2 AP7361C-33SP-13, U3 ESP32-C3-WROOM-02, U4 TPD4E05U06DQA, U5 SHT4x, U6 STCC4-D1, U7 AHT20_C2757850, U8 SGP40-D-R4, U9 ICP-20100

Commit message: Quicksave
Parts:
- moved U1 35.8 mm to (68.1, 31.9), turned to 0 degrees
- moved C2 31.9 mm to (64.0, 31.9), turned to 90 degrees
- moved R2 28.0 mm to (68.0, 34.5), turned to 0 degrees
- moved C6 12.9 mm to (51.5, 39.0), turned to 0 degrees
- moved R8 3.64 mm to (61.5, 35.0), turned to 180 degrees
- moved R7 2.62 mm to (64.5, 35.0), turned to 180 degrees
- moved C3 0.14 mm to (71.5, 36.5)
- moved C4 0.14 mm to (71.5, 34.5)
Routing:
- net VBUS: track 58.8 -> 96.0 mm
- net Net-(U1-STAT): track 12.7 -> 30.8 mm, vias 0 -> 2
- net +3V3: track 125.7 -> 108.4 mm
- net GND: track 90.2 -> 100.5 mm, vias 30 -> 32
- net /EN_VBAT: track 67.3 -> 61.5 mm
- net /VBAT: track 87.6 -> 91.2 mm
- net Net-(U1-PROG): track 10.1 -> 7.29 mm, vias 2 -> 0
- net /VBAT_DIV: track 27.8 -> 25.8 mm, vias 2 -> 4

Commit message: Separated PCBs
Parts:
- added C10: 4.7µF, Capacitor_SMD:C_0805_2012Metric, F.Cu at (98.5, 41.5)
- added J3: Conn_01x04, Connector_JST:JST_SH_SM04B-SRSS-TB_1x04-1MP_P1.00mm_Horizontal, F.Cu at (44.5, 34.0)
- added J4: Conn_01x04, Connector_JST:JST_SH_SM04B-SRSS-TB_1x04-1MP_P1.00mm_Horizontal, F.Cu at (95.0, 37.4)
- moved C9 57.3 mm to (98.0, 50.5), turned to 0 degrees
- moved U5 56.3 mm to (97.5, 48.0)
- moved C8 54.0 mm to (98.0, 53.0)
- moved R6 53.1 mm to (92.5, 41.5), turned to 0 degrees
- moved U7 51.8 mm to (93.0, 54.0)
- moved U8 50.6 mm to (92.5, 44.0)
- moved U9 50.1 mm to (96.0, 44.0)
- moved C7 50.1 mm to (98.5, 45.0), turned to -90 degrees
- moved U6 47.6 mm to (93.0, 49.0)
- moved D2 3.51 mm to (33.0, 32.5)
- moved R3 2.57 mm to (39.5, 37.5), turned to -90 degrees
Connections:
- C7 pad 1: +3V3 -> +3V3_EXT
- C7 pad 2: GND -> GND_EXT
- C8 pad 1: +3V3 -> +3V3_EXT
- C8 pad 2: GND -> GND_EXT
- C9 pad 1: +3V3 -> +3V3_EXT
- C9 pad 2: GND -> GND_EXT
- R6 pad 2: +3V3 -> +3V3_EXT
- U5 pad 3: +3V3 -> +3V3_EXT
- U5 pad 4: GND -> GND_EXT
- U6 pad 1: /SCL -> /SCL_EXT
- U6 pad 3: +3V3 -> +3V3_EXT
- U6 pad 4: GND -> GND_EXT
- U6 pad 5: /SDA -> /SDA_EXT
- U6 pad 6: +3V3 -> +3V3_EXT
- U6 pad 7: +3V3 -> +3V3_EXT
- U7 pad 2: +3V3 -> +3V3_EXT
- U7 pad 3: /SCL -> /SCL_EXT
- U7 pad 4: /SDA -> /SDA_EXT
- U7 pad 5: GND -> GND_EXT
- U8 pad 2: GND -> GND_EXT
- U8 pad 3: /SDA -> /SDA_EXT
- U8 pad 4: GND -> GND_EXT
- U8 pad 5: +3V3 -> +3V3_EXT
- U8 pad 6: /SCL -> /SCL_EXT
- U8 pad 7: GND -> GND_EXT
- U9 pad 1: +3V3 -> +3V3_EXT
- U9 pad 10: +3V3 -> +3V3_EXT
- U9 pad 2: /SCL -> /SCL_EXT
- U9 pad 3: GND -> GND_EXT
- U9 pad 4: /SDA -> /SDA_EXT
- U9 pad 5: +3V3 -> +3V3_EXT
- U9 pad 6: GND -> GND_EXT
- U9 pad 8: GND -> GND_EXT
- U9 pad 9: GND -> GND_EXT
Routing:
- net +3V3_EXT: track 0.00 -> 54.1 mm, vias 0 -> 4
- net GND: track 100.5 -> 56.9 mm, vias 32 -> 27
- net GND_EXT: track 0.00 -> 43.4 mm, vias 0 -> 7
- net +3V3: track 108.4 -> 76.2 mm, vias 10 -> 8
- net /SDA_EXT: track 0.00 -> 31.7 mm, vias 0 -> 5
- net /SCL_EXT: track 0.00 -> 24.3 mm, vias 0 -> 3
- net VBUS: track 96.0 -> 78.3 mm, vias 6 -> 4
- net /SCL: track 53.5 -> 38.9 mm, vias 5 -> 0
- net /SDA: track 52.9 -> 41.0 mm, vias 5 -> 4
- net Net-(U1-STAT): track 30.8 -> 34.8 mm, vias 2 -> 4
- net Net-(U5-SCL): track 7.84 -> 5.56 mm, vias 0 -> 2
- net Net-(D2-K): track 5.75 -> 6.96 mm
- net Net-(U5-SDA): track 6.27 -> 5.43 mm, vias 0 -> 2
Other:
- board size 50 x 35 mm -> 70 x 35 mm

Commit message: Battery fuel gauge
Parts:
- added C11: 470nF, Capacitor_SMD:C_0805_2012Metric, F.Cu at (40.0, 58.5)
- added C12: 1µF, Capacitor_SMD:C_0805_2012Metric, F.Cu at (39.5, 55.5)
- added R11: 0.01Ω, Resistor_SMD:R_0805_2012Metric, F.Cu at (55.9, 42.5)
- added R12: 10kΩ, Resistor_SMD:R_0805_2012Metric, F.Cu at (48.0, 60.0)
- added R13: 10kΩ, Resistor_SMD:R_0805_2012Metric, F.Cu at (49.5, 56.5)
- added U10: BQ27441-G1, Package_SON:Texas_S-PDSO-N12, F.Cu at (44.6, 56.8)
Connections:
- J2 pad 1: /VBAT -> /VBAT_PRE
Routing:
- net /VBAT_PRE: track 0.00 -> 40.6 mm, vias 0 -> 4
- net /VBAT: track 91.2 -> 112.9 mm, vias 3 -> 7
- net /SDA: track 41.0 -> 57.7 mm, vias 4 -> 5
- net Net-(U10-V_{DD}): track 0.00 -> 14.5 mm, vias 0 -> 2
- net /SCL: track 38.9 -> 50.4 mm, vias 0 -> 2
- net GND: track 56.9 -> 68.4 mm, vias 27 -> 28
- net Net-(U10-BIN): track 0.00 -> 5.25 mm
- net Net-(U10-GPOUT): track 0.00 -> 3.05 mm
- net /USB_D-: track 75.4 -> 77.1 mm
