File: Kicad/ambient-air.kicad_pcb (KiCad board)
At the start: 2 copper layers, 65.1 x 35 mm, 49 parts, among them J1 USB_C_Receptacle_USB2.0_14P, J2 Conn_01x02, J3 Conn_01x04, J4 Conn_01x04, SW1 SW_Push, SW2 MINI MSK12CO2, SW3 SW_Push, U1 MCP73831T-2ACI/MC, U10 BQ27441-G1, U2 AP7361C-33SP-13, U3 ESP32-C3-WROOM-02, U4 TPD4E05U06DQA, U5 SHT4x, U6 STCC4-D1, U7 AHT20_C2757850, U8 SGP40-D-R4, U9 ICP-20100

Commit message: Progress
Connections:
- R10 pad 2: Net-(J1-CC1) -> Net-(J1-CC2)
- R9 pad 2: Net-(J1-CC2) -> Net-(J1-CC1)
- SW1 pad 2: Net-(U3-EN/CHIP_PU) -> Net-(U3-GPIO4/ADC1_CH4)
- U3 pad 3: unconnected-(U3-GPIO4/ADC1_CH4-Pad3) -> Net-(U3-GPIO4/ADC1_CH4)
Routing:
- net Net-(U3-GPIO4/ADC1_CH4): track 0.00 -> 37.4 mm, vias 0 -> 4
- net Net-(U3-EN/CHIP_PU): track 36.2 -> 27.8 mm, vias 4 -> 2
- net Net-(J1-CC1): track 11.0 -> 7.09 mm
- net Net-(J1-CC2): track 10.1 -> 8.12 mm, vias 2 -> 0
Other:
- board text added: "Rev 3"
Changed lines of the file:
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@@
 	(net 30 "/SCL")
 	(net 31 "/SDA")
-	(net 32 "unconnected-(U3-GPIO4{slash}ADC1_CH4-Pad3)")
+	(net 32 "Net-(U3-GPIO4{slash}ADC1_CH4)")
 	(net 33 "unconnected-(U3-GPIO0{slash}ADC1_CH0{slash}XTAL_32K_P-Pad18)")
 	(net 34 "Net-(U3-GPIO3{slash}ADC1_CH3)")
@@
 			(size 1.5 0.9)
 			(layers "F.Cu" "F.Mask" "F.Paste")
-			(net 32 "unconnected-(U3-GPIO4{slash}ADC1_CH4-Pad3)")
+			(net 32 "Net-(U3-GPIO4{slash}ADC1_CH4)")
 			(pinfunction "GPIO4/ADC1_CH4")
-			(pintype "bidirectional+no_connect")
+			(pintype "bidirectional")
 		)
 		(pad "4" smd rect
@@
 			(layers "F.Cu" "F.Mask" "F.Paste")
 			(roundrect_rratio 0.243902)
-			(net 11 "Net-(J1-CC2)")
+			(net 9 "Net-(J1-CC1)")
 			(pintype "passive")
 		)
@@
 			(layers "F.Cu" "F.Mask" "F.Paste")
 			(roundrect_rratio 0.243902)
-			(net 9 "Net-(J1-CC1)")
+			(net 11 "Net-(J1-CC2)")
 			(pintype "passive")
 		)
@@
 			(size 2.42 1.28)
 			(layers "F.Cu" "F.Mask" "F.Paste")
-			(net 13 "Net-(U3-EN{slash}CHIP_PU)")
+			(net 32 "Net-(U3-GPIO4{slash}ADC1_CH4)")
 			(pinfunction "2")
 			(pintype "passive")
@@
 		(layer "Edge.Cuts")
 	)
-	(gr_text "Rev 2"
+	(gr_text "Rev 3"
 		(at 75 64 0)
 		(layer "F.SilkS")
@@
 	)
 	(segment
-		(start 33.826 54.0865)
-		(end 32.9125 55)
+		(start 33.3125 41.2)
+		(end 33.3125 42.3125)
+		(width 0.2)
+		(layer "F.Cu")
+		(net 9)
+	)
+	(segment
+		(start 35.629 45.107824)
+		(end 36.771176 46.25)
 		(width 0.2)
 		(layer "F.Cu")
@@
 	)
 	(segment
-		(start 33.826 49.128076)
-		(end 33.826 54.0865)
+		(start 35.629 44.629)
+		(end 35.629 45.107824)
 		(width 0.2)
 		(layer "F.Cu")
@@
 	)
 	(segment
-		(start 36.704076 46.25)
-		(end 33.826 49.128076)
+		(start 36.771176 46.25)
+		(end 37.38 46.25)
 		(width 0.2)
 		(layer "F.Cu")
@@
 	)
 	(segment
-		(start 37.38 46.25)
-		(end 36.704076 46.25)
+		(start 33.3125 42.3125)
+		(end 35.629 44.629)
 		(width 0.2)
 		(layer "F.Cu")
@@
 	)
 	(segment
-		(start 35.452773 46.652773)
-		(end 35.452773 44.252773)
+		(start 32.9125 54.3)
+		(end 35 52.2125)
 		(width 0.2)
 		(layer "F.Cu")
@@
 	)
 	(segment
-		(start 37.38 49.25)
-		(end 36.771176 49.25)
+		(start 36.488992 49.25)
+		(end 37.38 49.25)
 		(width 0.2)
 		(layer "F.Cu")
@@
 	)
 	(segment
-		(start 33.3125 42.1125)
-		(end 33.3125 41.2)
+		(start 35 50.738992)
+		(end 36.488992 49.25)
 		(width 0.2)
 		(layer "F.Cu")
@@
 	)
 	(segment
-		(start 36.771176 49.25)
-		(end 35.997746 48.47657)
+		(start 32.9125 55)
+		(end 32.9125 54.3)
 		(width 0.2)
 		(layer "F.Cu")
@@
 	)
 	(segment
-		(start 35.997746 48.47657)
-		(end 35.997746 47.804859)
+		(start 35 52.2125)
+		(end 35 50.738992)
 		(width 0.2)
 		(layer "F.Cu")
@@
 	)
 	(segment
-		(start 35.452773 44.252773)
-		(end 33.3125 42.1125)
-		(width 0.2)
-		(layer "F.Cu")
-		(net 11)
-	)
-	(via
-		(at 35.997746 47.804859)
-		(size 0.6)
-		(drill 0.3)
-		(layers "F.Cu" "B.Cu")
-		(net 11)
-	)
-	(via
-		(at 35.452773 46.652773)
-		(size 0.6)
-		(drill 0.3)
-		(layers "F.Cu" "B.Cu")
-		(net 11)
-	)
-	(segment
-		(start 35.997746 47.804859)
-		(end 35.997746 47.197746)
-		(width 0.2)
-		(layer "B.Cu")
-		(net 11)
-	)
-	(segment
-		(start 35.997746 47.197746)
-		(end 35.452773 46.652773)
-		(width 0.2)
-		(layer "B.Cu")
-		(net 11)
-	)
-	(segment
 		(start 59.95962 60.54038)
 		(end 59.298 61.202)
@@
 	)
 	(segment
-		(start 52.4 54.8875)
-		(end 54.2 56.6875)
-		(width 0.2)
-		(layer "F.Cu")
-		(net 13)
-	)
-	(segment
-		(start 54.2 56.6875)
-		(end 54.2 56.8)
-		(width 0.2)
-		(layer "F.Cu")
-		(net 13)
-	)
-	(segment
 		(start 55.4 52.199)
 		(end 61.161689 52.199)
@@
 	)
 	(segment
-		(start 56.2 60)
-		(end 57.9 60)
-		(width 0.2)
-		(layer "F.Cu")
-		(net 13)
-	)
-	(segment
 		(start 64.724 48.636689)
 		(end 64.724 45.076)
@@
 	)
 	(segment
-		(start 54.8 58.6)
-		(end 56.2 60)
-		(width 0.2)
-		(layer "F.Cu")
-		(net 13)
-	)
-	(segment
 		(start 52.4 54.8875)
 		(end 52.9115 54.8875)
@@
 	)
 	(via
-		(at 54.2 56.8)
-		(size 0.6)
-		(drill 0.3)
-		(layers "F.Cu" "B.Cu")
-		(net 13)
-	)
-	(via
-		(at 54.8 58.6)
-		(size 0.6)
-		(drill 0.3)
-		(layers "F.Cu" "B.Cu")
-		(net 13)
-	)
-	(via
 		(at 55.4 52.199)
 		(size 0.6)
@@
 	)
 	(segment
-		(start 54.2 56.8)
-		(end 54.2 58)
-		(width 0.2)
-		(layer "B.Cu")
-		(net 13)
-	)
-	(segment
 		(start 54.4 53.199)
 		(end 55.4 52.199)
@@
 	)
 	(segment
-		(start 54.2 58)
-		(end 54.8 58.6)
-		(width 0.2)
-		(layer "B.Cu")
-		(net 13)
-	)
-	(segment
 		(start 54.4 53.399)
 		(end 54.4 53.199)
@@
 	)
 	(segment
-		(start 57.2 57.8)
-		(end 57.4 57.6)
-		(width 0.2)
-		(layer "F.Cu")
-		(net 31)
-	)
-	(segment
 		(start 51.147711 43.580611)
 		(end 45 37.4329)
@@
 	)
 	(segment
+		(start 56 57.8)
+		(end 52.6 57.8)
+		(width 0.2)
+		(layer "F.Cu")
+		(net 31)
+	)
+	(segment
 		(start 42.725 55.7625)
 		(end 42.725 55.225)
@@
 	)
 	(segment
-		(start 52.6 57.8)
-		(end 57.2 57.8)
-		(width 0.2)
-		(layer "F.Cu")
-		(net 31)
-	)
-	(segment
 		(start 53.279938 52.024732)
 		(end 53.279938 44.067748)
@@
 	)
 	(via
-		(at 57.4 57.6)
+		(at 56 57.8)
 		(size 0.6)
 		(drill 0.3)
@@
 	)
 	(segment
+		(start 53.279938 57.120062)
+		(end 52.6 57.8)
+		(width 0.2)
+		(layer "B.Cu")
+		(net 31)
+	)
+	(segment
+		(start 56.2 57.6)
+		(end 61.304913 57.6)
+		(width 0.2)
+		(layer "B.Cu")
+		(net 31)
+	)
+	(segment
 		(start 61.304913 57.6)
 		(end 61.654913 57.25)
@@
 	)
 	(segment
-		(start 53.279938 57.120062)
-		(end 52.6 57.8)
+		(start 56 57.8)
+		(end 56.2 57.6)
 		(width 0.2)
 		(layer "B.Cu")
@@
 	)
 	(segment
-		(start 57.4 57.6)
-		(end 61.304913 57.6)
+		(start 69.55 36.689337)
+		(end 69.675 36.814337)
+		(width 0.2)
+		(layer "F.Cu")
+		(net 32)
+	)
+	(segment
+		(start 57.9 60)
+		(end 57.569 59.669)
+		(width 0.2)
+		(layer "F.Cu")
+		(net 32)
+	)
+	(segment
+		(start 57.569 59.669)
+		(end 57.569 54.41984)
+		(width 0.2)
+		(layer "F.Cu")
+		(net 32)
+	)
+	(segment
+		(start 70.275 50)
+		(end 70.275 41.275)
+		(width 0.2)
+		(layer "F.Cu")
+		(net 32)
+	)
+	(segment
+		(start 69.675 36.814337)
+		(end 69.675 38.75)
+		(width 0.2)
+		(layer "F.Cu")
+		(net 32)
+	)
+	(segment
+		(start 70.275 41.275)
+		(end 70 41)
+		(width 0.2)
+		(layer "F.Cu")
+		(net 32)
+	)
+	(segment
+		(start 57.569 54.41984)
+		(end 57.98884 54)
+		(width 0.2)
+		(layer "F.Cu")
+		(net 32)
+	)
+	(segment
+		(start 57.98884 54)
+		(end 60 54)
+		(width 0.2)
+		(layer "F.Cu")
+		(net 32)
+	)
+	(via
+		(at 69.55 36.689337)
+		(size 0.6)
+		(drill 0.3)
+		(layers "F.Cu" "B.Cu")
+		(net 32)
+	)
+	(via
+		(at 70 41)
+		(size 0.6)
+		(drill 0.3)
+		(layers "F.Cu" "B.Cu")
+		(net 32)
+	)
+	(via
+		(at 70.275 50)
+		(size 0.6)
+		(drill 0.3)
+		(layers "F.Cu" "B.Cu")
+		(net 32)
+	)
+	(via
+		(at 60 54)
+		(size 0.6)
+		(drill 0.3)
+		(layers "F.Cu" "B.Cu")
+		(net 32)
+	)
+	(segment
+		(start 70 41)
+		(end 70 37.139337)
 		(width 0.2)
 		(layer "B.Cu")
-		(net 31)
+		(net 32)
+	)
+	(segment
+		(start 60 51.650057)
+		(end 60.775321 50.874736)
+		(width 0.2)
+		(layer "B.Cu")
+		(net 32)
+	)
+	(segment
+		(start 60.775321 50.874736)
+		(end 69.400264 50.874736)
+		(width 0.2)
+		(layer "B.Cu")
+		(net 32)
+	)
+	(segment
+		(start 69.400264 50.874736)
+		(end 70.275 50)
+		(width 0.2)
+		(layer "B.Cu")
+		(net 32)
+	)
+	(segment
+		(start 70 37.139337)
+		(end 69.55 36.689337)
+		(width 0.2)
+		(layer "B.Cu")
+		(net 32)
+	)
+	(segment
+		(start 60 54)
+		(end 60 51.650057)
+		(width 0.2)
+		(layer "B.Cu")
+		(net 32)
 	)
 	(segment

Commit message: Get basic sampling working
Parts:
- removed JP1: Jumper_2_Open, Jumper:SolderJumper-2_P1.3mm_Open_TrianglePad1.0x1.5mm
- removed R7: 12kΩ, Resistor_SMD:R_0603_1608Metric
- removed R8: 10kΩ, Resistor_SMD:R_0603_1608Metric
- added R16: 668kΩ, Resistor_SMD:R_0603_1608Metric, F.Cu at (46.0, 42.0)
- added R17: 220kΩ, Resistor_SMD:R_0603_1608Metric, F.Cu at (40.0, 41.0)
- added U11: TPS2116DRL, Package_TO_SOT_SMD:SOT-583-8, F.Cu at (42.4, 40.5)
Connections:
- C1 pad 1: /VBAT -> /VDEV
- SW2 pad 3: /VBAT -> /VDEV
- U2 pad 8: /VBAT -> /VDEV
- U3 pad 16: /VBAT_DIV -> /PWR_SRC
Routing:
- net /VDEV: track 0.00 -> 80.7 mm, vias 0 -> 8
- net /VBAT: track 112.9 -> 58.2 mm, vias 7 -> 3
- net /PWR_SRC: track 0.00 -> 52.4 mm, vias 0 -> 6
- net /VBAT_DIV: track 25.8 -> 0.00 mm, vias 4 -> 0
- net VBUS: track 78.3 -> 90.0 mm
- net Net-(U11-PR1): track 0.00 -> 6.06 mm
- net GND: track 68.4 -> 70.1 mm
- net +3V3: track 76.2 -> 76.9 mm
- added copper zone on F.Cu, net /VDEV
Other:
- board text added: "Rev 4"
- board text removed: "Rev 3"
