File: Kicad/ambient-air.kicad_sch (KiCad schematic)
At the start: 47 parts, among them J1 USB_C_Receptacle_USB2.0_14P, J2 Conn_01x02, J3 Conn_01x04, J4 Conn_01x04, SW1 SW_Push, SW2 MINI MSK12CO2, SW3 SW_Push, U1 MCP73831T-2ACI/MC, U10 BQ27441-G1, U11 TPS2116DRL, U2 AP7361C-33SP-13, U3 ESP32-C3-WROOM-02, U4 TPD4E05U06DQA, U5 SHT4x, U6 STCC4-D1, U7 AHT20_C2757850, U8 SGP40-D-R4, U9 ICP-20100

Commit message: Add RTC to pcb and move sgp40 from sensor to main pcb
Parts:
- added C10, C15: 1µF, Capacitor_SMD:C_0603_1608Metric, symbol Device:C_Small
- added C11: 100nF, Capacitor_SMD:C_0805_2012Metric, symbol Device:C_Small
- added U9: RX8111CE, easyeda2kicad:OSC-SMD_10P-L3.2-W2.5-BL-1, symbol easyeda2kicad:RX8111CE
- C1, C9: footprint Capacitor_SMD:C_0805_2012Metric -> Capacitor_SMD:C_0603_1608Metric
- C7: renamed from C12; footprint Capacitor_SMD:C_0805_2012Metric -> Capacitor_SMD:C_0603_1608Metric
- renumbered C10 to C12, C8 to C13, C7 to C14, C11 to C8, J3 to J1, J1 to J2, J2 to J3, R13 to R10, R17 to R11, R16 to R12, R6 to R13, R12 to R6, R11 to R7, R10 to R8, SW2 to SW1, SW3 to SW2, SW1 to SW3, U9 to U10, U7 to U11, U6 to U12, U10 to U5, U11 to U6, U8 to U7, U5 to U8
Connections:
- net +3V3: now also C9.1, R13.2, U7.5 (VDDH), U9.8 (VIO)
- net +3V3_EXT: no longer C9.1, R13.2, U7.5 (VDDH)
- net GND: now also C9.2, U7.2 (VSS), U7.4 (N/A), U7.7 (EXP), C10.2, C11.2, C15.2, U9.6 (EVIN), U9.9 (GND)
- net GND_EXT: no longer C9.2, U7.2 (VSS), U7.4 (N/A), U7.7 (EXP)
- net SCL: now also U7.6 (SCL), U9.5 (SCL)
- net SCL_EXT: no longer U7.6 (SCL)
- net SDA: now also U7.3 (SDA), U9.7 (SDA)
- net SDA_EXT: no longer U7.3 (SDA)
- net VBAT: now also C11.1, U9.1 (VDD), U9.3 (VBAT)
- net at R13.1, U7.1 (VDD): now also C15.1
- net TIME_INT: now reaches U3.18 (GPIO0/ADC1_CH0/XTAL_32K_P)
- net TIME_INT: now also U9.10 (/INT)
- new net: C10.1, U9.2 (VOUT)
Other:
- note added: "I2C Address: 0x32"
- moved on the sheet: C9, R13, U7
