File: Kicad/boards/main.kicad_pcb (KiCad board)
At the start: 2 copper layers, 50 x 35 mm, 37 parts, among them J1 USB_C_Receptacle_USB2.0_14P, J2 Conn_01x02, J3 Conn_01x04, SW1 SW_Push, SW2 MINI MSK12CO2, SW3 SW_Push, U1 MCP73831T-2ACI/MC, U10 BQ27441-G1, U2 AP7361C-33SP-13, U3 ESP32-C3-WROOM-02, U4 TPD4E05U06DQA

Commit message: Progress
Connections:
- R10 pad 2: Net-(J1-CC1) -> Net-(J1-CC2)
- R9 pad 2: Net-(J1-CC2) -> Net-(J1-CC1)
- SW1 pad 2: Net-(U3-EN/CHIP_PU) -> Net-(U3-GPIO4/ADC1_CH4)
- U3 pad 3: unconnected-(U3-GPIO4/ADC1_CH4-Pad3) -> Net-(U3-GPIO4/ADC1_CH4)
Routing:
- net Net-(U3-GPIO4/ADC1_CH4): track 0.00 -> 37.4 mm, vias 0 -> 4
- net Net-(U3-EN/CHIP_PU): track 36.2 -> 27.8 mm, vias 4 -> 2
- net Net-(J1-CC1): track 11.0 -> 7.09 mm
- net Net-(J1-CC2): track 10.1 -> 8.12 mm, vias 2 -> 0
Other:
- board text added: "Rev 3"
- board text removed: "Rev 2"

Commit message: Get basic sampling working
Parts:
- removed JP1: Jumper_2_Open, Jumper:SolderJumper-2_P1.3mm_Open_TrianglePad1.0x1.5mm
- removed R7: 12kΩ, Resistor_SMD:R_0603_1608Metric
- removed R8: 10kΩ, Resistor_SMD:R_0603_1608Metric
- added R16: 668kΩ, Resistor_SMD:R_0603_1608Metric, F.Cu at (139.5, 32.0)
- added R17: 220kΩ, Resistor_SMD:R_0603_1608Metric, F.Cu at (133.5, 31.0)
- added U11: TPS2116DRL, Package_TO_SOT_SMD:SOT-583-8, F.Cu at (135.9, 30.5)
Connections:
- C1 pad 1: /VBAT -> /VDEV
- SW2 pad 3: /VBAT -> /VDEV
- U2 pad 8: /VBAT -> /VDEV
- U3 pad 16: /VBAT_DIV -> /PWR_SRC
Routing:
- net /VDEV: track 0.00 -> 80.7 mm, vias 0 -> 8
- net /VBAT: track 112.9 -> 58.2 mm, vias 7 -> 3
- net /PWR_SRC: track 0.00 -> 52.4 mm, vias 0 -> 6
- net /VBAT_DIV: track 25.8 -> 0.00 mm, vias 4 -> 0
- net VBUS: track 78.3 -> 90.0 mm
- net Net-(U11-PR1): track 0.00 -> 6.06 mm
- net GND: track 68.4 -> 70.1 mm
- net +3V3: track 76.2 -> 76.9 mm
- added copper zone on F.Cu, net /VDEV
Other:
- board text added: "Rev 4"
- board text removed: "Rev 3"
